File: DistBoard/distboard/distboard.sch (KiCad schematic (older format))
At the start: 11 parts

Commit message: Playing with dist board PCB
Parts:
- F1: renamed from F?; footprint (none) -> Fuse_Holders_and_Fuses:BladeFuse-Mini
- J1: renamed from J?; footprint (none) -> Connectors_WAGO:WAGO_734_2pin_Straight_RuggedPads
- J2: renamed from J?; footprint (none) -> Connectors_Molex:Molex_KK-6410-02_02x2.54mm_Straight
- J3: renamed from J?; footprint (none) -> Connectors:USB_A_Vertical
- J4, J5, J6, J7, J8: renamed from J?; footprint (none) -> Connectors:RJ45_8
- U1: renamed from U?; footprint (none) -> mini360:MINI-360
- gave numbers to parts that had none: 1
Changed lines of the file:
@@
 EESchema Schematic File Version 4
+LIBS:distboard-cache
 EELAYER 26 0
 EELAYER END
@@
 $EndDescr
 $Comp
-L Connector:RJ45_Shielded J?
+L Connector:RJ45_Shielded J4
 U 1 1 5B60B297
 P 3450 850
-F 0 "J?" V 3200 1350 50  0000 L CNN
+F 0 "J4" V 3200 1350 50  0000 L CNN
 F 1 "CAN_1" H 3350 1400 50  0000 L CNN
-F 2 "" V 3450 875 50  0001 C CNN
+F 2 "Connectors:RJ45_8" V 3450 875 50  0001 C CNN
 F 3 "~" V 3450 875 50  0001 C CNN
 	1    3450 850
@@
 $EndComp
 $Comp
-L power:+24V #PWR?
+L power:+24V #PWR01
 U 1 1 5B60B47E
 P 850 1700
-F 0 "#PWR?" H 850 1550 50  0001 C CNN
+F 0 "#PWR01" H 850 1550 50  0001 C CNN
 F 1 "+24V" H 865 1873 50  0000 C CNN
 F 2 "" H 850 1700 50  0001 C CNN
@@
 $EndComp
 $Comp
-L Connector:Screw_Terminal_01x02 J?
+L Connector:Screw_Terminal_01x02 J1
 U 1 1 5B60B4E3
 P 850 700
-F 0 "J?" V 816 512 50  0000 R CNN
+F 0 "J1" V 816 512 50  0000 R CNN
 F 1 "POWER_IN" V 950 800 50  0000 R CNN
-F 2 "" H 850 700 50  0001 C CNN
+F 2 "Connectors_WAGO:WAGO_734_2pin_Straight_RuggedPads" H 850 700 50  0001 C CNN
 F 3 "~" H 850 700 50  0001 C CNN
 	1    850  700
@@
 $EndComp
 $Comp
-L power:GND #PWR?
+L power:GND #PWR02
 U 1 1 5B60B5B6
 P 1000 950
-F 0 "#PWR?" H 1000 700 50  0001 C CNN
+F 0 "#PWR02" H 1000 700 50  0001 C CNN
 F 1 "GND" H 1005 777 50  0000 C CNN
 F 2 "" H 1000 950 50  0001 C CNN
@@
 CANL
 $Comp
-L power:GND #PWR?
+L power:GND #PWR012
 U 1 1 5B60B8B9
 P 2950 900
-F 0 "#PWR?" H 2950 650 50  0001 C CNN
+F 0 "#PWR012" H 2950 650 50  0001 C CNN
 F 1 "GND" H 2955 727 50  0000 C CNN
 F 2 "" H 2950 900 50  0001 C CNN
@@
 	2950 850  2950 900
 $Comp
-L Diode:1N5819 D?
+L Diode:1N5819 D1
 U 1 1 5B60B9F5
 P 850 1550
-F 0 "D?" V 896 1471 50  0000 R CNN
+F 0 "D1" V 896 1471 50  0000 R CNN
 F 1 "1N5819" V 805 1471 50  0000 R CNN
 F 2 "Diode_THT:D_DO-41_SOD81_P10.16mm_Horizontal" H 850 1375 50  0001 C CNN
@@
 $EndComp
 $Comp
-L Device:Fuse F?
+L Device:Fuse F1
 U 1 1 5B60BA80
 P 850 1250
-F 0 "F?" H 910 1296 50  0000 L CNN
+F 0 "F1" H 910 1296 50  0000 L CNN
 F 1 "Fuse" H 910 1205 50  0000 L CNN
-F 2 "" V 780 1250 50  0001 C CNN
+F 2 "Fuse_Holders_and_Fuses:BladeFuse-Mini" V 780 1250 50  0001 C CNN
 F 3 "~" H 850 1250 50  0001 C CNN
 	1    850  1250
@@
 	850  900  850  1100
 $Comp
-L Connector_Generic:Conn_01x02 J?
+L Connector_Generic:Conn_01x02 J2
 U 1 1 5B60C018
 P 1650 700
-F 0 "J?" V 1616 512 50  0000 R CNN
+F 0 "J2" V 1616 512 50  0000 R CNN
 F 1 "FAN_HEADER" V 1750 850 50  0000 R CNN
-F 2 "" H 1650 700 50  0001 C CNN
+F 2 "Connectors_Molex:Molex_KK-6410-02_02x2.54mm_Straight" H 1650 700 50  0001 C CNN
 F 3 "~" H 1650 700 50  0001 C CNN
 	1    1650 700
@@
 $EndComp
 $Comp
-L power:GND #PWR?
+L power:GND #PWR08
 U 1 1 5B60C0E9
 P 1750 900
-F 0 "#PWR?" H 1750 650 50  0001 C CNN
+F 0 "#PWR08" H 1750 650 50  0001 C CNN
 F 1 "GND" H 1755 727 50  0000 C CNN
 F 2 "" H 1750 900 50  0001 C CNN
@@
 $EndComp
 $Comp
-L Connector:RJ45_Shielded J?
+L Connector:RJ45_Shielded J6
 U 1 1 5B60C2F8
 P 4650 850
-F 0 "J?" V 4400 1350 50  0000 L CNN
+F 0 "J6" V 4400 1350 50  0000 L CNN
 F 1 "CAN_2" H 4550 1400 50  0000 L CNN
-F 2 "" V 4650 875 50  0001 C CNN
+F 2 "Connectors:RJ45_8" V 4650 875 50  0001 C CNN
 F 3 "~" V 4650 875 50  0001 C CNN
 	1    4650 850
@@
 CANL
 $Comp
-L power:GND #PWR?
+L power:GND #PWR014
 U 1 1 5B60C309
 P 4150 900
-F 0 "#PWR?" H 4150 650 50  0001 C CNN
+F 0 "#PWR014" H 4150 650 50  0001 C CNN
 F 1 "GND" H 4155 727 50  0000 C CNN
 F 2 "" H 4150 900 50  0001 C CNN
@@
 	4150 850  4150 900
 $Comp
-L Connector:RJ45_Shielded J?
+L Connector:RJ45_Shielded J7
 U 1 1 5B60C3A8
 P 5850 850
-F 0 "J?" V 5600 1350 50  0000 L CNN
+F 0 "J7" V 5600 1350 50  0000 L CNN
 F 1 "CAN_3" H 5750 1400 50  0000 L CNN
-F 2 "" V 5850 875 50  0001 C CNN
+F 2 "Connectors:RJ45_8" V 5850 875 50  0001 C CNN
 F 3 "~" V 5850 875 50  0001 C CNN
 	1    5850 850
@@
 CANL
 $Comp
-L power:GND #PWR?
+L power:GND #PWR016
 U 1 1 5B60C3B9
 P 5350 900
-F 0 "#PWR?" H 5350 650 50  0001 C CNN
+F 0 "#PWR016" H 5350 650 50  0001 C CNN
 F 1 "GND" H 5355 727 50  0000 C CNN
 F 2 "" H 5350 900 50  0001 C CNN
@@
 	5350 850  5350 900
 $Comp
-L Connector:RJ45_Shielded J?
+L Connector:RJ45_Shielded J8
 U 1 1 5B60C64E
 P 7050 850
-F 0 "J?" V 6800 1350 50  0000 L CNN
+F 0 "J8" V 6800 1350 50  0000 L CNN
 F 1 "CAN_4" H 6950 1400 50  0000 L CNN
-F 2 "" V 7050 875 50  0001 C CNN
+F 2 "Connectors:RJ45_8" V 7050 875 50  0001 C CNN
 F 3 "~" V 7050 875 50  0001 C CNN
 	1    7050 850
@@
 CANL
 $Comp
-L power:GND #PWR?
+L power:GND #PWR017
 U 1 1 5B60C65F
 P 6550 900
-F 0 "#PWR?" H 6550 650 50  0001 C CNN
+F 0 "#PWR017" H 6550 650 50  0001 C CNN
 F 1 "GND" H 6555 727 50  0000 C CNN
 F 2 "" H 6550 900 50  0001 C CNN
@@
 	6550 850  6550 900
 $Comp
-L Connector:RJ45_Shielded J?
+L Connector:RJ45_Shielded J5
 U 1 1 5B60C86F
 P 3850 2450
-F 0 "J?" V 3600 2950 50  0000 L CNN
+F 0 "J5" V 3600 2950 50  0000 L CNN
 F 1 "CAN_PI" H 3750 3000 50  0000 L CNN
-F 2 "" V 3850 2475 50  0001 C CNN
+F 2 "Connectors:RJ45_8" V 3850 2475 50  0001 C CNN
 F 3 "~" V 3850 2475 50  0001 C CNN
 	1    3850 2450
@@
 CANL
 $Comp
-L power:GND #PWR?
+L power:GND #PWR015
 U 1 1 5B60C880
 P 4350 2450
-F 0 "#PWR?" H 4350 2200 50  0001 C CNN
+F 0 "#PWR015" H 4350 2200 50  0001 C CNN
 F 1 "GND" H 4355 2277 50  0000 C CNN
 F 2 "" H 4350 2450 50  0001 C CNN
@@
 $EndComp
 $Comp
-L Connector:USB_A J?
+L Connector:USB_A J3
 U 1 1 5B60CFE8
 P 2800 2450
-F 0 "J?" H 2600 2250 50  0000 R CNN
+F 0 "J3" H 2600 2250 50  0000 R CNN
 F 1 "PI_POWER" V 2550 2750 50  0000 R CNN
-F 2 "" H 2950 2400 50  0001 C CNN
+F 2 "Connectors:USB_A_Vertical" H 2950 2400 50  0001 C CNN
 F 3 " ~" H 2950 2400 50  0001 C CNN
 	1    2800 2450
@@
 CANGND
 $Comp
-L power:+24V #PWR?
+L power:+24V #PWR05
 U 1 1 5B60ECBB
 P 1450 1450
-F 0 "#PWR?" H 1450 1300 50  0001 C CNN
+F 0 "#PWR05" H 1450 1300 50  0001 C CNN
 F 1 "+24V" H 1465 1623 50  0000 C CNN
 F 2 "" H 1450 1450 50  0001 C CNN
@@
 $EndComp
 $Comp
-L power:GND #PWR?
+L power:GND #PWR06
 U 1 1 5B60ED16
 P 1450 1550
-F 0 "#PWR?" H 1450 1300 50  0001 C CNN
+F 0 "#PWR06" H 1450 1300 50  0001 C CNN
 F 1 "GND" H 1455 1377 50  0000 C CNN
 F 2 "" H 1450 1550 50  0001 C CNN
@@
 	1450 1550 1500 1550
 $Comp
-L mini-360:MINI-360 U?
+L mini-360:MINI-360 U1
 U 1 1 5B60FBCE
 P 1750 2350
-F 0 "U?" H 1750 2625 50  0000 C CNN
+F 0 "U1" H 1750 2625 50  0000 C CNN
 F 1 "MINI-360" H 1750 2534 50  0000 C CNN
-F 2 "" H 1750 2350 50  0001 C CNN
+F 2 "mini360:MINI-360" H 1750 2350 50  0001 C CNN
 F 3 "" H 1750 2350 50  0001 C CNN
 	1    1750 2350
@@
 $EndComp
 $Comp
-L power:+24V #PWR?
+L power:+24V #PWR03
 U 1 1 5B60FD6B
 P 1400 2300
-F 0 "#PWR?" H 1400 2150 50  0001 C CNN
+F 0 "#PWR03" H 1400 2150 50  0001 C CNN
 F 1 "+24V" H 1415 2473 50  0000 C CNN
 F 2 "" H 1400 2300 50  0001 C CNN
@@
 $EndComp
 $Comp
-L power:GND #PWR?
+L power:GND #PWR04
 U 1 1 5B60FDA2
 P 1400 2450
-F 0 "#PWR?" H 1400 2200 50  0001 C CNN
+F 0 "#PWR04" H 1400 2200 50  0001 C CNN
 F 1 "GND" H 1405 2277 50  0000 C CNN
 F 2 "" H 1400 2450 50  0001 C CNN
@@
 $EndComp
 $Comp
-L power:+5V #PWR?
+L power:+5V #PWR09
 U 1 1 5B60FDE8
 P 2100 2300
-F 0 "#PWR?" H 2100 2150 50  0001 C CNN
+F 0 "#PWR09" H 2100 2150 50  0001 C CNN
 F 1 "+5V" H 2115 2473 50  0000 C CNN
 F 2 "" H 2100 2300 50  0001 C CNN
@@
 $EndComp
 $Comp
-L power:GND #PWR?
+L power:GND #PWR010
 U 1 1 5B60FE10
 P 2100 2450
-F 0 "#PWR?" H 2100 2200 50  0001 C CNN
+F 0 "#PWR010" H 2100 2200 50  0001 C CNN
 F 1 "GND" H 2105 2277 50  0000 C CNN
 F 2 "" H 2100 2450 50  0001 C CNN
@@
 $EndComp
 $Comp
-L power:+5V #PWR?
+L power:+5V #PWR011
 U 1 1 5B60FE31
 P 2350 2650
-F 0 "#PWR?" H 2350 2500 50  0001 C CNN
+F 0 "#PWR011" H 2350 2500 50  0001 C CNN
 F 1 "+5V" H 2365 2823 50  0000 C CNN
 F 2 "" H 2350 2650 50  0001 C CNN
@@
 	2350 2650 2500 2650
 $Comp
-L power:GND #PWR?
+L power:GND #PWR013
 U 1 1 5B61033F
 P 3200 2050
-F 0 "#PWR?" H 3200 1800 50  0001 C CNN
+F 0 "#PWR013" H 3200 1800 50  0001 C CNN
 F 1 "GND" H 3205 1877 50  0000 C CNN
 F 2 "" H 3200 2050 50  0001 C CNN
@@
 Connection ~ 2900 2050
 $Comp
-L power:+5V #PWR?
+L power:+5V #PWR07
 U 1 1 5B610B3A
 P 1600 900
-F 0 "#PWR?" H 1600 750 50  0001 C CNN
+F 0 "#PWR07" H 1600 750 50  0001 C CNN
 F 1 "+5V" H 1615 1073 50  0000 C CNN
 F 2 "" H 1600 900 50  0001 C CNN
