File: Hardware/DistBoard/distboard.sch (KiCad schematic (older format))
At the start: 11 parts, among them J1 POWER_IN, J2 FAN_HEADER, J3 PI_POWER, J4 CAN_1, J5 CAN_PI, J6 CAN_2, J7 CAN_3, J8 CAN_4, U1 MINI-360

Commit message: Working on dist board
Parts:
- removed J3: PI_POWER, Connectors:USB_A_Vertical, symbol Connector:USB_A
- added C1: 100uF, Capacitor_Tantalum_SMD:CP_EIA-3528-21_Kemet-B_Pad1.50x2.35mm_HandSolder, symbol Device:CP
- added C2: 10uF, Capacitor_SMD:C_0603_1608Metric_Pad1.05x0.95mm_HandSolder, symbol Device:C
- added MH1, MH2, MH3, MH4: MountingHole_Pad, MountingHole:MountingHole_3.2mm_M3_Pad_Via, symbol Mechanical:MountingHole_Pad
- added U2, U3, U4: double_usb, Connector_USB:USB_A_Wuerth_61400826021_Horizontal_Stacked, symbol stacked_usb:double_usb
- J1: footprint Connectors_WAGO:WAGO_734_2pin_Straight_RuggedPads -> Connector_Wago:Wago_734-162_1x02_P3.50mm_Horizontal
- J4, J5, J6, J7, J8: footprint Connectors:RJ45_8 -> RJ45:RJ45_GENERIC
Connections:
- wire segments 33 -> 48
Other:
- moved on the sheet: J5

Commit message: Finished distboard design
Parts:
- added D?: POWER, LED_SMD:LED_0805_2012Metric_Pad1.15x1.40mm_HandSolder, symbol Device:LED
- added R?: 1K, Resistor_SMD:R_0603_1608Metric_Pad1.05x0.95mm_HandSolder, symbol Device:R
Changed lines of the file:
@@
 Wire Wire Line
 	3250 3200 3450 3200
+$Comp
+L Device:LED D?
+U 1 1 5B722C3A
+P 800 2400
+F 0 "D?" V 838 2282 50  0000 R CNN
+F 1 "POWER" V 747 2282 50  0000 R CNN
+F 2 "LED_SMD:LED_0805_2012Metric_Pad1.15x1.40mm_HandSolder" H 800 2400 50  0001 C CNN
+F 3 "~" H 800 2400 50  0001 C CNN
+	1    800  2400
+	0    -1   -1   0
+$EndComp
+$Comp
+L Device:R R?
+U 1 1 5B722C9F
+P 800 2700
+F 0 "R?" H 870 2746 50  0000 L CNN
+F 1 "1K" H 870 2655 50  0000 L CNN
+F 2 "Resistor_SMD:R_0603_1608Metric_Pad1.05x0.95mm_HandSolder" V 730 2700 50  0001 C CNN
+F 3 "~" H 800 2700 50  0001 C CNN
+	1    800  2700
+	1    0    0    -1
+$EndComp
+$Comp
+L power:GND #PWR?
+U 1 1 5B722F1D
+P 800 2850
+F 0 "#PWR?" H 800 2600 50  0001 C CNN
+F 1 "GND" H 805 2677 50  0000 C CNN
+F 2 "" H 800 2850 50  0001 C CNN
+F 3 "" H 800 2850 50  0001 C CNN
+	1    800  2850
+	1    0    0    -1
+$EndComp
+$Comp
+L power:+5V #PWR?
+U 1 1 5B722F52
+P 800 2250
+F 0 "#PWR?" H 800 2100 50  0001 C CNN
+F 1 "+5V" H 815 2423 50  0000 C CNN
+F 2 "" H 800 2250 50  0001 C CNN
+F 3 "" H 800 2250 50  0001 C CNN
+	1    800  2250
+	1    0    0    -1
+$EndComp
 $EndSCHEMATC
